File: arduinotask.kicad_pcb (KiCad board)
At the start: 2 copper layers, 12 parts, among them J1 5V IN, SW1 1825910-2, SW2 1825910-2, U1 ATmega328-P, U2 LCD-016N002L, Y1 16MHz

Commit message: second commit
Parts:
- moved R3 33.3 mm to (48.1, 70.5)
Connections:
- SW1 pad 3: /RESET -> unconnected-(SW1-Pad3)
- U1 pad 22: Net-(U1-GND-Pad22) -> GND
- U1 pad 7: unconnected-(U1-VCC-Pad7) -> +5V
- U1 pad 8: Net-(U1-GND-Pad22) -> GND
Routing:
- net /IN1: track 6.50 -> 48.0 mm
- net /rs: track 0.00 -> 38.1 mm, vias 0 -> 2
- net GND: track 166.1 -> 202.9 mm
- net /e: track 0.00 -> 33.0 mm
- net /d7: track 0.00 -> 15.0 mm
- net /d4: track 0.00 -> 14.9 mm
- net /d6: track 0.00 -> 12.1 mm
- net +5V: track 112.3 -> 124.0 mm
- net /d5: track 0.00 -> 11.2 mm
- net Net-(U2-VO): track 0.00 -> 10.6 mm
- net Net-(U1-GND-Pad22): track 8.67 -> 0.00 mm
